File: eagle/tuner.brd (EAGLE design)
At the start: 42.8 x 53.3 mm, 58 parts, among them IC1 MEGA8-AI, IC2 LM358D, Q2 BSS123, Q3 SST5485, Q4 BSS123, U1 LP2985AIM5-5.0, U2 LP2985AIM5-5.0

Commit message: work on next revision PCB
Parts:
- removed D1: BAT54, diode:SOT23
- removed L1: 10uH, inductor-neosid:SM-1206
- removed L2: 33uH, rcl:6000-XXXX-RC
- removed Q2, Q4: BSS123, transistor-small-signal:SOT23
- removed Q3: SST5485, transistor-fet:SOT23
- removed U$1: IRF9389TRPBF, IRF9389TRPBF:SO08
- added C19, C26: 1u, eagle-ltspice:C0805
- added C21, C24, C27: 0.1uF, eagle-ltspice:C0805
- added C25: 1uF, eagle-ltspice:C0805
- added D2: BAS40-04, diode:SOT23
- added IC3: LM358D, linear:SO08
- added PASS, VOL: (no value), pinhead:1X02
- added R15, R23: 1k, resistor:M0805
- added R21, R22: 10k, resistor:M0805
- added R24, R25: 100k, resistor:M0805
- added TP1, TP2, TP3: PTR1B1,27, testpad:B1,27
- added U3: ADC121S021CIMF, ADC121S021CIMF:SOT95P284X122-6N
- C10: value 47uF -> 96n; device rcl:E2-5 -> eagle-ltspice:C0805
- C12: value 2.2uF -> 1uF
- C14: value 0.1uF -> 47n
- C15: value 1uF -> 47n
- C16: value 2.2uF -> 47n
- C17: value 470pF -> 47n
- C20: value 470uF -> 0.1uF; device rcl:E3,5-8 -> eagle-ltspice:C0805
- R10: value 3k -> 68k
- R11: value 24k -> 34k
- R12: value 50k -> 0
- R13: value 1k -> 0
- R14: value 1k -> 259k
- R2: value 22M -> 10k
- R20: value 10k -> 1k
- R3: value 11M -> 10M
- R4: value 10k -> 259k
- R5: value 11M -> 10k
- R8: value 50k -> 68k; device rcl:RTRIM4G/J -> resistor:M0805
- R9: value 27k -> 100k
- U2: value LP2985AIM5-5.0 -> SSM2305RMZ-R2; device LP2985AIM5-5.0:SOT95P284X119-5N -> SSM2305RMZ-R2:SOP65P490X110-8N
- moved R20 342.7 mm to (11.4, -281.9), turned to 0 degrees
- moved C20 274.8 mm to (11.4, -203.2), turned to 0 degrees
- moved C12 239.7 mm to (11.4, -171.4)
- moved C17 189.3 mm to (20.3, -115.6)
- moved C16 185.6 mm to (20.3, -109.2)
- moved R14 178.7 mm to (20.3, -128.3), turned to 0 degrees
- moved R4 178.5 mm to (20.3, -121.9)
- moved U2 168.3 mm to (22.9, -94.0)
- moved C15 150.0 mm to (20.3, -71.1)
- moved R13 142.2 mm to (20.3, -83.8), turned to 0 degrees
- moved R12 138.0 mm to (20.3, -77.5), turned to 0 degrees
- moved R11 122.6 mm to (20.3, -58.4), turned to 0 degrees
- moved C14 116.2 mm to (20.3, -64.8), turned to 0 degrees
- moved R10 110.9 mm to (20.3, -45.7), turned to 0 degrees
- moved C10 107.6 mm to (20.3, -52.1), turned to 0 degrees
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Connections:
- net N$8 renamed MOSI
- removed net 2.5V: C16.1, IC2.3, Q3.2, R20.2, R5.1, U2.5
- removed net N$1: C4.2, IC1.18, L1.2
- removed net N$33: Q3.3, Q4.3, R20.1
- removed net N$34: C17.1, U2.4
- new net BUZZER: IC1.1, R25.1, VOL.2
- new net CS_ADC: IC1.24, U3.6
- new net MISO: IC1.16, SV1.6, U3.5
- new net N$8: C12.2, IC3.3, IC3.5, R21.2, R22.1
- new net SCK: IC1.17, SV1.4, U3.4
- new net SD_AMP: IC1.32, U2.1
- net 5V: now also C20.2, C21.2, C24.2, C27.2, C4.2, D2.2, IC1.18, IC3.8, R2.1, R21.1, U2.6, U3.1; no longer L1.1
- net 9V: no longer C11.1, R4.2, U$1.7, U$1.8, U2.1, U2.3
- net GND: now also C10.1, C11.1, C12.1, C20.1, C21.1, C24.1, C27.1, D2.1, IC3.4, PASS.1, R11.1, R12.2, R22.2, R5.2, U2.7, U3.2; no longer C10.-, C11.2, C12.2, C14.1, C17.2, IC1.14, OUT.1, Q2.2, U$1.5, U$1.6
- net N$10: now also C14.1, R24.1, R8.2, R9.1, TP1.TP; no longer C15.1, R2.2, R9.2
- net N$11: now also OUT.2, U2.8; no longer L2.1, U$1.1, U$1.3
- net N$13: now also R15.1, R9.2; no longer R2.1
- net N$14: now also R4.2, U2.3; no longer C12.1, C20.+, L2.2
- net N$15: now also C25.2, PASS.2; no longer C14.2, IC1.23, R14.1
- net N$16: now also D2.3
- net N$17: now also C11.2, R15.2, R2.2, R5.1; no longer C15.2, R5.2
- net N$18: now also C25.1, C26.1, IC3.1, R20.2; no longer IC1.1, Q2.1
- net N$19: now also C14.2, C15.1, R11.2; no longer IC2.2, R10.2, R9.1
- net N$20: now also C15.2, IC2.3; no longer Q3.1, R11.2
- net N$21: now also R14.2, U2.4; no longer C20.-, OUT.2
- net N$27: now also C10.2, R10.2, R8.1; no longer D1.1, IC2.1, R11.1, R14.2
- net N$29: now also C16.1, R14.1; no longer C10.+, D1.3, R8.3
- net N$30: now also IC2.1, IC2.2, R13.2, TP2.TP, U3.3; no longer R12.2, R8.1
- net N$31: now also C17.1, R4.1; no longer Q4.1, R8.2
- net N$32: now also C26.2, IC3.2, R20.1, R24.2, R25.2; no longer Q4.2, R13.2
- net N$6: now also C17.2, C19.1, IC3.7, R23.2, TP3.TP; no longer IC1.16, SV1.6
- net N$7: now also C19.2, IC3.6, R23.1, VOL.1; no longer IC1.17, SV1.4
- net N$9: now also OUT.1, U2.5; no longer Q2.3, R4.1, U$1.2, U$1.4
Routing:
- net 2.5V: track 40.2 -> 0.00 mm, vias 2 -> 0
- net N$27: track 28.6 -> 0.00 mm
- net SCK: track 0.00 -> 20.5 mm, vias 0 -> 1
- net N$7: track 20.5 -> 0.00 mm, vias 1 -> 0
- net N$9: track 17.3 -> 0.00 mm
- net N$6: track 16.1 -> 0.00 mm, vias 1 -> 0
- net MISO: track 0.00 -> 16.1 mm, vias 0 -> 1
- net N$29: track 14.6 -> 0.00 mm
- net N$11: track 11.7 -> 0.00 mm
- net N$14: track 10.9 -> 0.00 mm
- net N$1: track 9.46 -> 0.00 mm
- net N$19: track 9.40 -> 0.00 mm
- net N$33: track 9.09 -> 0.00 mm
- net N$20: track 8.53 -> 0.00 mm
- net 9V: track 36.5 -> 28.6 mm
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
Commit message: do board layout
Parts:
- added C28: 0.1u, eagle-ltspice:C0805
- moved R24 353.7 mm to (48.3, 63.5), turned to 180 degrees
- moved R25 351.3 mm to (34.3, 55.9), turned to 90 degrees
- moved C27 350.1 mm to (49.5, 47.0)
- moved R20 342.1 mm to (45.7, 58.4), turned to 180 degrees
- moved C26 339.4 mm to (44.5, 62.2), turned to 90 degrees
- moved C25 326.8 mm to (44.5, 55.9), turned to 180 degrees
- moved PASS 314.3 mm to (38.1, 55.9)
- moved C21 306.6 mm to (54.6, 63.5), turned to 90 degrees
- moved C24 303.7 mm to (52.1, 54.6), turned to 90 degrees
- moved VOL 286.0 mm to (30.5, 57.1), turned to 270 degrees
- moved TP2 276.9 mm to (57.1, 58.4)
- moved TP3 275.9 mm to (25.4, 55.9)
- moved C20 269.3 mm to (38.1, 64.8)
- moved TP1 256.3 mm to (61.0, 41.9)
- moved R23 255.7 mm to (26.7, 58.4), turned to 180 degrees
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Connections:
- new net FG: C10.1, R11.1, R12.2, R13.1
- new net N$1: C28.1, R24.1
- net BUZZER: now also IC1.13; no longer IC1.1
- net GND: no longer C10.1, R11.1, R12.2, R13.1
- net N$10: now also C28.2; no longer R24.1
- net SD_AMP: now also IC1.1; no longer IC1.32
Routing:
- net 5V: track 96.0 -> 188.9 mm, vias 0 -> 1
- net N$10: track 8.10 -> 45.7 mm, vias 0 -> 3
- net SD_AMP: track 0.00 -> 30.7 mm
- net MISO: track 16.1 -> 39.6 mm, vias 1 -> 2
- net BUZZER: track 0.00 -> 21.8 mm
- net N$32: track 0.00 -> 21.1 mm
- net N$20: track 0.00 -> 20.0 mm
- net N$6: track 0.00 -> 20.0 mm
- net SCK: track 20.5 -> 38.6 mm, vias 1 -> 2
- net N$8: track 0.00 -> 17.4 mm, vias 0 -> 2
- net CS_ADC: track 0.00 -> 17.2 mm, vias 0 -> 2
- net 9V: track 28.6 -> 13.0 mm
- net N$7: track 0.00 -> 13.8 mm
- net FG: track 0.00 -> 13.4 mm, vias 0 -> 2
- net N$17: track 1.90 -> 14.3 mm
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
Commit message: lemme smash
Routing:
- net N$10: track 45.7 -> 44.6 mm
- net N$19: track 5.59 -> 4.45 mm
- net MOSI: track 24.2 -> 23.3 mm
